Commit message: synchronize urdf and rviz robots

File: isaacpjt/cobot3/urdf/cobot3.urdf (robot description, URDF)
Before this commit: robot cobot3, 16 links, 15 joints
Links:
- removed link rear_pivot_link
- removed link rear_wheel_link
- added link caster_frame_base, mass 0.8
- added link caster_swivel_left, mass 0.3; visual mesh filename=file:///home/rokey/cobot3_ws/isaacpjt/cobot3/meshes/carter/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
- added link caster_swivel_right, mass 0.3; visual mesh filename=file:///home/rokey/cobot3_ws/isaacpjt/cobot3/meshes/carter/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
- added link caster_wheel_left, mass 0.6; visual mesh filename=file:///home/rokey/cobot3_ws/isaacpjt/cobot3/meshes/carter/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
- added link caster_wheel_right, mass 0.6; visual mesh filename=file:///home/rokey/cobot3_ws/isaacpjt/cobot3/meshes/carter/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
- link chassis_link: geometry collision box size=.55 .40 .54; visual mesh filename=file:///home/rokey/cobot3_ws/isaacpjt/cobot3/meshes/carter/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
- link left_wheel_link: geometry collision cylinder length=0.1 radius=0.240; visual mesh filename=file:///home/rokey/cobot3_ws/isaacpjt/cobot3/meshes/carter/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
- link m0609_base_link: geometry collision mesh filename=file:///home/rokey/cobot3_ws/isaacpjt/cobot3/meshes/m0609/m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 scale=0.001 0.001 0.001; visual mesh filename=file:///home/rokey/cobot3_ws/isaacpjt/cobot3/meshes/m0609/m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 scale=0.001 0.001 0.001
- link m0609_link_1: geometry collision mesh filename=file:///home/rokey/cobot3_ws/isaacpjt/cobot3/meshes/m0609/m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 scale=0.001 0.001 0.001; visual mesh filename=file:///home/rokey/cobot3_ws/isaacpjt/cobot3/meshes/m0609/m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 scale=0.001 0.001 0.001
- link m0609_link_2: geometry collision mesh filename=file:///home/rokey/cobot3_ws/isaacpjt/cobot3/meshes/m0609/m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 scale=0.001 0.001 0.001; collision mesh filename=file:///home/rokey/cobot3_ws/isaacpjt/cobot3/meshes/m0609/m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 scale=0.001 0.001 0.001
- link m0609_link_3: geometry collision mesh filename=file:///home/rokey/cobot3_ws/isaacpjt/cobot3/meshes/m0609/m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 scale=0.001 0.001 0.001; visual mesh filename=file:///home/rokey/cobot3_ws/isaacpjt/cobot3/meshes/m0609/m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 scale=0.001 0.001 0.001
- link m0609_link_4: geometry collision mesh filename=file:///home/rokey/cobot3_ws/isaacpjt/cobot3/meshes/m0609/m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 scale=0.001 0.001 0.001; collision mesh filename=file:///home/rokey/cobot3_ws/isaacpjt/cobot3/meshes/m0609/m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 scale=0.001 0.001 0.001
- link m0609_link_5: geometry collision mesh filename=file:///home/rokey/cobot3_ws/isaacpjt/cobot3/meshes/m0609/m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 scale=0.001 0.001 0.001; visual mesh filename=file:///home/rokey/cobot3_ws/isaacpjt/cobot3/meshes/m0609/m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 scale=0.001 0.001 0.001
- link m0609_link_6: geometry collision mesh filename=file:///home/rokey/cobot3_ws/isaacpjt/cobot3/meshes/m0609/m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 scale=0.001 0.001 0.001; visual mesh filename=file:///home/rokey/cobot3_ws/isaacpjt/cobot3/meshes/m0609/m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 scale=0.001 0.001 0.001
- link right_wheel_link: geometry collision cylinder length=0.1 radius=0.240; visual mesh filename=file:///home/rokey/cobot3_ws/isaacpjt/cobot3/meshes/carter/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
Joints:
- removed joint rear_axle
- removed joint rear_pivot
- added joint joint_caster_base: type revolute, parent chassis_link, child caster_frame_base, origin xyz=-0.47195 0 0.22289 rpy=-1.5707963 0 1.5707963, axis 0 0 1, limit lower=-2.0 upper=2.0 effort=1000 velocity=10.0
- added joint joint_caster_left: type continuous, parent caster_swivel_left, child caster_wheel_left, origin xyz=-0.115397885 -0.000050042 0.039999098 rpy=-1.5707963 1.5707963 0, axis 0 0 1
- added joint joint_caster_right: type continuous, parent caster_swivel_right, child caster_wheel_right, origin xyz=-0.11539289 0.000050033 0.03999913 rpy=-1.5707963 1.5707963 0, axis 0 0 1
- added joint joint_swing_left: type continuous, parent caster_frame_base, child caster_swivel_left, origin xyz=0.132296 0.031188007 0.000001991 rpy=0 0 -1.5707963, axis 1 0 0
- added joint joint_swing_right: type continuous, parent caster_frame_base, child caster_swivel_right, origin xyz=-0.1323 0.031187888 0.000000114 rpy=0 0 -1.5707963, axis 1 0 0
